File: board/DIYPie.kicad_pcb (KiCad board)
At the start: 6 copper layers, 87.2 x 79.2 mm, 42 parts, among them J1 DF40C-100DS-0.4V(51), J2 DF40C-100DS-0.4V(51), J3 CUI_DEVICES_SJ-43514-SMT, J4 MOLEX_5033981892, J5 MOLEX_2137160001, Q1 EMH2T2R, Q2 EMH2T2R, SW1 POWER, SW2 VOL_UP, SW3 VOL_DOWN, U1 TPS65132W, U2 TPS61176, U3 TPS61023, U4 TLV320AIC3110IRHB

Commit message: Migrated to 5.99 (and other changes)
Parts:
- removed DS1: LPM035M407B, DIYPie:245863050104829+
- removed H1, H2, H3, H4: Hole, MountingHole:MountingHole_2.2mm_M2
- removed J5: MOLEX_2137160001, DIYPie:MOLEX_2137160001
- removed Q1, Q2: EMH2T2R, DIYPie:SOT-563
- removed R2: 82K, DIYPie:R_0402_1005Metric_InvertedHomeplate
- removed XA1: CM4, DIYPie:CM4_LowProfile_NoHoles
- added C1001: 4u7, DIYPie:C_0603_1608Metric, F.Cu at (61.4, 115.6)
- added C1002: 4u7, DIYPie:C_0603_1608Metric, F.Cu at (67.3, 111.4)
- added C1003: 0u1, DIYPie:C_0402_1005Metric, F.Cu at (64.7, 122.6)
- added C1004: 0u1, DIYPie:C_0402_1005Metric, F.Cu at (61.1, 126.7)
- added C1005: 470n, DIYPie:C_0402_1005Metric, F.Cu at (73.1, 114.7)
- added C1006: 0u1, DIYPie:C_0402_1005Metric, F.Cu at (85.6, 103.6)
- added C1007: 0u1, DIYPie:C_0402_1005Metric, F.Cu at (81.5, 110.0)
- added C1008: 470n, DIYPie:C_0402_1005Metric, F.Cu at (76.6, 111.1)
- added C1009: 0u1, DIYPie:C_0402_1005Metric, F.Cu at (77.0, 114.0)
- added C1010: 0u1, DIYPie:C_0402_1005Metric, F.Cu at (85.6, 106.5)
- added C1011: 10u, DIYPie:C_0603_1608Metric, F.Cu at (76.2, 104.1)
- added C1012: 10u, DIYPie:C_0603_1608Metric, F.Cu at (63.9, 115.6)
- added C1013: 10u, DIYPie:C_0603_1608Metric, F.Cu at (61.4, 119.6)
- added C1014: 10u, DIYPie:C_0603_1608Metric, F.Cu at (67.3, 115.4)
- added C1015: 47u, DIYPie:C_0805_2012Metric, F.Cu at (64.5, 111.4)
- added C1016: 470p, DIYPie:C_0402_1005Metric, F.Cu at (87.5, 103.6)
- added C1017: 470p, DIYPie:C_0402_1005Metric, F.Cu at (61.1, 129.6)
- added C1018: 47n, DIYPie:C_0402_1005Metric, F.Cu at (81.5, 107.1)
- added C1019: 470n, DIYPie:C_0402_1005Metric, F.Cu at (67.2, 121.8)
- added C1020: 47u, DIYPie:C_0805_2012Metric, F.Cu at (61.6, 111.4)
- added C1021: 470p, DIYPie:C_0402_1005Metric, F.Cu at (83.5, 107.1)
- added C1022: 470p, DIYPie:C_0402_1005Metric, F.Cu at (73.1, 117.6)
- added C1023: 47n, DIYPie:C_0402_1005Metric, F.Cu at (79.5, 110.0)
- added C1101: 1u, DIYPie:C_0402_1005Metric, F.Cu at (155.7, 34.1)
- added C1102: 1u, DIYPie:C_0402_1005Metric, F.Cu at (148.8, 41.7)
- added C1103: 470n, DIYPie:C_0402_1005Metric, F.Cu at (157.7, 34.1)
- added C1104: 4u7, DIYPie:C_0603_1608Metric, F.Cu at (153.5, 34.6)
- added C1105: 4u7, DIYPie:C_0805_2012Metric, F.Cu at (145.5, 45.0)
- added C1201: 1u, DIYPie:C_0402_1005Metric, F.Cu at (109.4, 38.1)
- added C1202: 4u7, DIYPie:C_0603_1608Metric, F.Cu at (107.2, 34.6)
- added C1203: 4u7, DIYPie:C_0603_1608Metric, F.Cu at (101.9, 45.9)
- added C1204: 10u, DIYPie:C_0603_1608Metric, F.Cu at (109.7, 34.6)
- added C1205: 10u, DIYPie:C_0603_1608Metric, F.Cu at (101.9, 49.9)
- added C1206: 10u, DIYPie:C_0603_1608Metric, F.Cu at (107.2, 38.6)
- added C1301: 1u, DIYPie:C_0402_1005Metric, F.Cu at (17.7, 117.8)
- added C15: 10u, DIYPie:C_0603_1608Metric, F.Cu at (51.8, 162.5)
- added C1501: 470n, DIYPie:C_0402_1005Metric, F.Cu at (172.5, 150.9)
- added C1502: 10u, DIYPie:C_0603_1608Metric, F.Cu at (170.3, 151.5)
- added C16: 10u, DIYPie:C_0603_1608Metric, F.Cu at (38.5, 175.3)
- added C1601: 0u1, DIYPie:C_0402_1005Metric, F.Cu at (290.8, 45.6)
- added C1602: 470n, DIYPie:C_0402_1005Metric, F.Cu at (301.3, 34.1)
- added C17: 220p, DIYPie:C_0402_1005Metric, F.Cu at (34.3, 169.3)
- added C1701: 470n, DIYPie:C_0402_1005Metric, F.Cu at (193.3, 92.5)
- added C1702: 470n, DIYPie:C_0402_1005Metric, F.Cu at (191.3, 98.3)
- added C1703: 470n, DIYPie:C_0402_1005Metric, F.Cu at (191.3, 92.5)
- added C18: 0u1, DIYPie:C_0402_1005Metric, F.Cu at (46.0, 172.3)
- added C1802: 4u7, DIYPie:C_0603_1608Metric, F.Cu at (152.7, 157.0)
- added C1803: 220p, DIYPie:C_0402_1005Metric, F.Cu at (152.5, 164.5)
- added C1804: 10u, DIYPie:C_0603_1608Metric, F.Cu at (152.7, 161.0)
- added C1805: 10u, DIYPie:C_0603_1608Metric, F.Cu at (158.3, 151.5)
- added C19: 220p, DIYPie:C_0402_1005Metric, F.Cu at (41.1, 184.9)
- added C20: 470n, DIYPie:C_0402_1005Metric, F.Cu at (45.0, 179.0)
- added C201: 1u, DIYPie:C_0402_1005Metric, F.Cu at (251.6, 66.9)
- added C202: 1u, DIYPie:C_0402_1005Metric, F.Cu at (241.1, 74.3)
- added C203: 470n, DIYPie:C_0402_1005Metric, F.Cu at (235.9, 67.7)
- added C204: 4u7, DIYPie:C_0603_1608Metric, F.Cu at (238.6, 68.3)
- added C205: 1u, DIYPie:C_0402_1005Metric, F.Cu at (240.9, 71.4)
- added C206: 4u7, DIYPie:C_0603_1608Metric, F.Cu at (238.6, 72.3)
- added C207: 4u7, DIYPie:C_0805_2012Metric, F.Cu at (252.0, 63.2)
- added C208: 4u7, DIYPie:C_0603_1608Metric, F.Cu at (236.1, 72.0)
- added C209: 10u, DIYPie:C_0603_1608Metric, F.Cu at (243.9, 68.0)
- added C21: 10u, DIYPie:C_0603_1608Metric, F.Cu at (43.0, 168.8)
- added C210: 10u, DIYPie:C_0603_1608Metric, F.Cu at (246.4, 68.0)
- added C2101: 1u, DIYPie:C_0402_1005Metric, F.Cu at (198.6, 116.6)
- added C2102: 12p, DIYPie:C_0402_1005Metric, F.Cu at (198.6, 119.6)
- added C2103: 12p, DIYPie:C_0402_1005Metric, F.Cu at (200.6, 116.6)
- added C2104: 1u, DIYPie:C_0402_1005Metric, F.Cu at (191.3, 127.0)
- added C211: 10u, DIYPie:C_0603_1608Metric, F.Cu at (241.4, 68.0)
- added C22: 10u, DIYPie:C_0603_1608Metric, F.Cu at (36.0, 175.3)
- added C23: 0u1, DIYPie:C_0402_1005Metric, F.Cu at (155.0, 156.5)
- added C24: 0u1, DIYPie:C_0402_1005Metric, F.Cu at (237.0, 99.7)
- added C25: 0u1, DIYPie:C_0402_1005Metric, F.Cu at (233.1, 99.7)
- added C26: 0u1, DIYPie:C_0402_1005Metric, F.Cu at (235.0, 102.7)
- added C27: 1u, DIYPie:C_0402_1005Metric, F.Cu at (264.5, 66.0)
- added C28: 10u, DIYPie:C_0603_1608Metric, F.Cu at (276.1, 50.7)
- added C29: 47n, DIYPie:C_0402_1005Metric, F.Cu at (278.3, 50.1)
- added C30: 4u7, DIYPie:C_0603_1608Metric, F.Cu at (271.1, 50.7)
- added C31: 10u, DIYPie:C_0603_1608Metric, F.Cu at (264.8, 62.5)
- added C32: 10u, DIYPie:C_0603_1608Metric, F.Cu at (271.1, 54.7)
- added C33: 10u, DIYPie:C_0603_1608Metric, F.Cu at (273.6, 50.7)
- added C34: 220p, DIYPie:C_0402_1005Metric, F.Cu at (208.9, 123.4)
- added C35: 1u, DIYPie:C_0402_1005Metric, F.Cu at (212.7, 116.6)
- added C36: 220p, DIYPie:C_0402_1005Metric, F.Cu at (208.9, 120.5)
- added C401: 4u7, DIYPie:C_0603_1608Metric, F.Cu at (124.5, 165.4)
- added C402: 0u1, DIYPie:C_0402_1005Metric, F.Cu at (122.5, 168.8)
- added C403: 4u7, DIYPie:C_0603_1608Metric, F.Cu at (115.3, 170.6)
- added C404: 0u1, DIYPie:C_0402_1005Metric, F.Cu at (132.1, 162.2)
- added C405: 470n, DIYPie:C_0402_1005Metric, F.Cu at (135.2, 158.2)
- added C406: 0u1, DIYPie:C_0402_1005Metric, F.Cu at (119.5, 172.4)
- added C407: 0u1, DIYPie:C_0402_1005Metric, F.Cu at (117.5, 172.4)
- added C408: 470n, DIYPie:C_0402_1005Metric, F.Cu at (128.8, 164.9)
- added C409: 0u1, DIYPie:C_0402_1005Metric, F.Cu at (142.0, 150.9)
- added C410: 0u1, DIYPie:C_0402_1005Metric, F.Cu at (126.8, 164.8)
- added C411: 10u, DIYPie:C_0603_1608Metric, F.Cu at (117.8, 168.9)
- added C412: 10u, DIYPie:C_0603_1608Metric, F.Cu at (120.3, 168.9)
- added C413: 10u, DIYPie:C_0603_1608Metric, F.Cu at (132.9, 158.7)
- added C414: 10u, DIYPie:C_0603_1608Metric, F.Cu at (130.4, 158.6)
- added C415: 47u, DIYPie:C_0805_2012Metric, F.Cu at (127.7, 158.8)
- added C416: 47u, DIYPie:C_0805_2012Metric, F.Cu at (112.5, 170.8)
- added C417: 470n, DIYPie:C_0402_1005Metric, F.Cu at (130.8, 165.1)
- added C418: 47n, DIYPie:C_0402_1005Metric, F.Cu at (137.2, 158.2)
- added C419: 47n, DIYPie:C_0402_1005Metric, F.Cu at (144.0, 150.9)
- added C420: 470p, DIYPie:C_0402_1005Metric, F.Cu at (126.5, 170.6)
- added C421: 470p, DIYPie:C_0402_1005Metric, F.Cu at (122.5, 171.7)
- added C422: 470p, DIYPie:C_0402_1005Metric, F.Cu at (126.8, 167.7)
- added C423: 470p, DIYPie:C_0402_1005Metric, F.Cu at (124.5, 168.8)
- added C424: 470n, DIYPie:C_0402_1005Metric, F.Cu at (60.1, 162.0)
- added C425: 470n, DIYPie:C_0402_1005Metric, F.Cu at (55.8, 167.8)
- added C426: 470n, DIYPie:C_0402_1005Metric, F.Cu at (46.9, 177.6)
- added C427: 0u1, DIYPie:C_0402_1005Metric, F.Cu at (41.0, 179.0)
- added C428: 0u1, DIYPie:C_0402_1005Metric, F.Cu at (42.7, 176.1)
- added C429: 0u1, DIYPie:C_0402_1005Metric, F.Cu at (44.7, 176.1)
- added C501: 1u, DIYPie:C_0402_1005Metric, F.Cu at (239.1, 75.7)
- added D101: XBP1010-G, DIYPie:D_SOD-923, F.Cu at (276.4, 34.0)
- added D1101: PMEG4010CEJ, DIYPie:D_SOD-323F, F.Cu at (150.7, 35.0)
- added D1601: DF2B7AFS, DIYPie:D_SOD-923, F.Cu at (296.0, 40.9)
- added D201: PMEG4010CEJ, DIYPie:D_SOD-323F, F.Cu at (249.1, 63.3)
- added D401: DF2B7AFS, DIYPie:D_SOD-923, F.Cu at (132.7, 165.0)
- added D402: DF2B7AFS, DIYPie:D_SOD-923, F.Cu at (142.0, 156.6)
- added D403: DF2B7AFS, DIYPie:D_SOD-923, F.Cu at (134.7, 163.9)
- added D404: DF2B7AFS, DIYPie:D_SOD-923, F.Cu at (130.7, 167.9)
- added D405: DF2B7AFS, DIYPie:D_SOD-923, F.Cu at (144.0, 153.7)
- added D406: DF2B7AFS, DIYPie:D_SOD-923, F.Cu at (137.1, 161.0)
- added D407: DF2B7AFS, DIYPie:D_SOD-923, F.Cu at (146.0, 153.7)
- added D408: STATUS, DIYPie:KINGBRIGHT_APBA3010, F.Cu at (26.2, 179.3)
- added D701: DF2B7AFS, DIYPie:D_SOD-923, F.Cu at (151.5, 99.4)
- added D702: DF2B7AFS, DIYPie:D_SOD-923, F.Cu at (147.9, 102.9)
- added D801: DF2B7AFS, DIYPie:D_SOD-923, F.Cu at (192.0, 40.9)
- added D802: DF2B7AFS, DIYPie:D_SOD-923, F.Cu at (188.4, 44.5)
- added D901: DF2B7AFS, DIYPie:D_SOD-923, F.Cu at (116.7, 96.0)
- added D902: DF2B7AFS, DIYPie:D_SOD-923, F.Cu at (108.0, 111.5)
- added D903: DF2B7AFS, DIYPie:D_SOD-923, F.Cu at (118.6, 96.0)
- added DS1301: LPM035M407B, DIYPie:KYOCERA_245863050104829+, F.Cu at (18.7, 109.2)
- added DS201: LPM035M407B, DIYPie:KYOCERA_245863050104829+, F.Cu at (232.9, 68.1)
- added FB1: 120R, DIYPie:L_0402_1005Metric, F.Cu at (39.0, 179.0)
- added FB1001: 120R, DIYPie:L_0402_1005Metric, F.Cu at (63.1, 126.7)
- added FB1002: 120R, DIYPie:L_0402_1005Metric, F.Cu at (75.1, 114.7)
- added FB1003: 120R, DIYPie:L_0402_1005Metric, F.Cu at (66.6, 124.7)
- added FB1004: 120R, DIYPie:L_0402_1005Metric, F.Cu at (69.2, 121.8)
- added FB1901: 120R, DIYPie:L_0402_1005Metric, F.Cu at (220.5, 92.5)
- added FB401: 120R, DIYPie:L_0402_1005Metric, F.Cu at (130.2, 162.0)
- added FB402: 120R, DIYPie:L_0402_1005Metric, F.Cu at (146.0, 150.9)
- added FB403: 120R, DIYPie:L_0402_1005Metric, F.Cu at (128.8, 167.8)
- added FB404: 120R, DIYPie:L_0402_1005Metric, F.Cu at (135.2, 161.1)
- added H101: Hole, MountingHole:MountingHole_2.2mm_M2, F.Cu at (266.5, 35.6)
- added H102: Hole, MountingHole:MountingHole_2.2mm_M2, F.Cu at (266.5, 41.6)
- added H103: Hole, MountingHole:MountingHole_2.2mm_M2, F.Cu at (272.4, 35.6)
- added H104: Hole, MountingHole:MountingHole_2.2mm_M2, F.Cu at (272.4, 41.6)
- added J1401: MOLEX_5033981892, DIYPie:MOLEX_5033981892, F.Cu at (238.6, 46.5)
- added J1601: BAT, DIYPie:MOLEX_533980267, F.Cu at (295.0, 35.6)
- added J301: DF40C-100DS-0.4V(51), DIYPie:HIROSE_DF40C-100DS-0.4V(51)_NoPads, F.Cu at (65.0, 44.6)
- added J302: DF40C-100DS-0.4V(51), DIYPie:HIROSE_DF40C-100DS-0.4V(51)_NoPads, F.Cu at (60.5, 44.6)
- added J401: SPK_R, DIYPie:MOLEX_533980267, F.Cu at (121.0, 152.4)
- added J403: HP, DIYPie:CUI_DEVICES_SJ-43514-SMT, F.Cu at (109.7, 159.8)
- added J601: MOLEX_5033981892, DIYPie:MOLEX_5033981892, F.Cu at (74.9, 174.4)
- added J701: SPK_R, DIYPie:MOLEX_533980267, F.Cu at (152.2, 94.0)
- added J801: SPK_R, DIYPie:MOLEX_533980267, F.Cu at (192.7, 35.6)
- added J901: HP, DIYPie:CUI_DEVICES_SJ-43514-SMT, F.Cu at (109.7, 101.3)
- added L1101: 4u7, DIYPie:L_1008_2520Metric, F.Cu at (145.9, 40.4)
- added L1201: 4u7, DIYPie:L_1008_2520Metric, F.Cu at (102.5, 41.4)
- added L1801: 1u, DIYPie:L_TYA4020, F.Cu at (154.2, 152.2)
- added L201: 4u7, DIYPie:L_1008_2520Metric, F.Cu at (242.0, 63.5)
- added L202: 4u7, DIYPie:L_1008_2520Metric, F.Cu at (245.7, 63.5)
- added L3: 1u, DIYPie:L_TYA4020, F.Cu at (266.3, 57.8)
- added NT1001: Net-Tie_2, DIYPie:NetTie-2_SMD_Pad1.5mm, F.Cu at (63.9, 103.9)
- added NT1002: Net-Tie_2, DIYPie:NetTie-2_SMD_Pad1.5mm, F.Cu at (63.9, 107.4)
- added NT401: Net-Tie_2, DIYPie:NetTie-2_SMD_Pad1.5mm, F.Cu at (107.3, 170.3)
- added NT402: Net-Tie_2, DIYPie:NetTie-2_SMD_Pad1.5mm, F.Cu at (130.0, 154.8)
- added NT403: Net-Tie_2, DIYPie:NetTie-2_SMD_Pad1.5mm, F.Cu at (130.0, 151.2)
- added NT404: Net-Tie_2, DIYPie:NetTie-2_SMD_Pad1.5mm, F.Cu at (119.5, 165.1)
- added R10: 10K, DIYPie:R_0402_1005Metric, F.Cu at (47.8, 168.9)
- added R1001: 100R, DIYPie:R_0402_1005Metric, F.Cu at (79.5, 107.1)
- added R1002: 2K2, DIYPie:R_0402_1005Metric, F.Cu at (69.2, 118.9)
- added R1003: 100R, DIYPie:R_0402_1005Metric, F.Cu at (67.2, 118.9)
- added R11: 100R, DIYPie:R_0402_1005Metric, F.Cu at (243.2, 92.5)
- added R1101: 34K, DIYPie:R_0402_1005Metric, F.Cu at (145.0, 51.6)
- added R1102: 82K, DIYPie:R_0402_1005Metric, F.Cu at (152.3, 38.8)
- added R1103: 732K, DIYPie:R_0402_1005Metric, F.Cu at (145.0, 48.7)
- added R1104: 34K, DIYPie:R_0402_1005Metric, F.Cu at (150.3, 38.8)
- added R12: 100K, DIYPie:R_0402_1005Metric, F.Cu at (235.0, 99.7)
- added R13: 100K, DIYPie:R_0402_1005Metric, F.Cu at (239.2, 92.5)
- added R14: 100K, DIYPie:R_0402_1005Metric, F.Cu at (233.1, 102.7)
- added R15: 10K, DIYPie:R_0402_1005Metric, F.Cu at (273.3, 54.2)
- added R1501: 732K, DIYPie:R_0402_1005Metric, F.Cu at (170.0, 158.0)
- added R16: 10K, DIYPie:R_0402_1005Metric, F.Cu at (270.1, 58.2)
- added R17: 100K, DIYPie:R_0402_1005Metric, F.Cu at (17.7, 90.5)
- added R1701: 732K, DIYPie:R_0402_1005Metric, F.Cu at (191.3, 95.4)
- added R18: 10K, DIYPie:R_0402_1005Metric, F.Cu at (214.7, 116.6)
- added R1801: 732K, DIYPie:R_0402_1005Metric, F.Cu at (158.0, 154.9)
- added R1802: 732K, DIYPie:R_0402_1005Metric, F.Cu at (157.0, 157.8)
- added R1803: 100K, DIYPie:R_0402_1005Metric, F.Cu at (160.0, 154.9)
- added R19: 732K, DIYPie:R_0402_1005Metric, F.Cu at (210.9, 120.5)
- added R201: 34K, DIYPie:R_0402_1005Metric, F.Cu at (237.1, 75.7)
- added R202: 82K, DIYPie:R_0402_1005Metric, F.Cu at (237.1, 78.6)
- added R203: 732K, DIYPie:R_0402_1005Metric, F.Cu at (243.1, 74.3)
- added R204: 34K, DIYPie:R_0402_1005Metric, F.Cu at (242.9, 71.4)
- added R2101: 34K, DIYPie:R_0402_1005Metric, F.Cu at (195.2, 123.9)
- added R401: 2K2, DIYPie:R_0402_1005Metric, F.Cu at (124.5, 171.7)
- added R402: 100R, DIYPie:R_0402_1005Metric, F.Cu at (142.0, 153.8)
- added R403: 100R, DIYPie:R_0402_1005Metric, F.Cu at (139.2, 158.2)
- added R404: 34K, DIYPie:R_0402_1005Metric, F.Cu at (50.0, 171.8)
- added R405: 732K, DIYPie:R_0402_1005Metric, F.Cu at (62.1, 162.0)
- added R406: 10K, DIYPie:R_0402_1005Metric, F.Cu at (51.8, 168.9)
- added R407: 10K, DIYPie:R_0402_1005Metric, F.Cu at (54.1, 162.0)
- added R408: 100K, DIYPie:R_0402_1005Metric, F.Cu at (49.8, 168.9)
- added R409: 10K, DIYPie:R_0402_1005Metric, F.Cu at (51.1, 166.0)
- added R410: 100R, DIYPie:R_0402_1005Metric, F.Cu at (21.5, 185.5)
- added R411: 100R, DIYPie:R_0402_1005Metric, F.Cu at (49.1, 166.0)
- added R412: 100K, DIYPie:R_0402_1005Metric, F.Cu at (56.1, 164.9)
- added R413: 100K, DIYPie:R_0402_1005Metric, F.Cu at (54.1, 164.9)
- added R414: 100K, DIYPie:R_0402_1005Metric, F.Cu at (39.0, 182.0)
- added R5: 10K, DIYPie:R_0402_1005Metric, F.Cu at (50.0, 174.7)
- added R6: 10K, DIYPie:R_0402_1005Metric, F.Cu at (39.1, 184.9)
- added R601: 732K, DIYPie:R_0402_1005Metric, F.Cu at (83.7, 166.0)
- added R7: 732K, DIYPie:R_0402_1005Metric, F.Cu at (35.7, 182.5)
- added R8: 732K, DIYPie:R_0402_1005Metric, F.Cu at (35.2, 185.5)
- added R9: 100K, DIYPie:R_0402_1005Metric, F.Cu at (58.1, 162.0)
- added SW401: POWER, DIYPie:CKCOMPONENTS_PTS845VM20PSMTR4LFS, F.Cu at (30.0, 173.5)
- added SW402: VOL-, DIYPie:CKCOMPONENTS_PTS845VM20PSMTR4LFS, F.Cu at (19.5, 180.5)
- added SW501: VOL+, DIYPie:CKCOMPONENTS_PTS845VM20PSMTR4LFS, F.Cu at (38.5, 164.2)
- added TP1001: TestPoint, DIYPie:TestPoint_Pad_D1.5mm, F.Cu at (70.3, 114.7)
- added TP1002: TestPoint, DIYPie:TestPoint_Pad_D1.5mm, F.Cu at (61.9, 123.4)
- added TP1003: TestPoint, DIYPie:TestPoint_Pad_D1.5mm, F.Cu at (82.8, 103.9)
- added TP1004: TestPoint, DIYPie:TestPoint_Pad_D1.5mm, F.Cu at (79.2, 103.9)
- added TP1005: TestPoint, DIYPie:TestPoint_Pad_D1.5mm, F.Cu at (70.3, 111.2)
- added TP1006: TestPoint, DIYPie:TestPoint_Pad_D1.5mm, F.Cu at (76.7, 107.9)
- added TP1007: TestPoint, DIYPie:TestPoint_Pad_D1.5mm, F.Cu at (64.4, 119.4)
- added TP1008: TestPoint, DIYPie:TestPoint_Pad_D1.5mm, F.Cu at (73.8, 111.5)
- added TP701: TestPoint, DIYPie:TestPoint_Pad_D1.5mm, F.Cu at (159.2, 92.8)
- added TP702: TestPoint, DIYPie:TestPoint_Pad_D1.5mm, F.Cu at (148.7, 99.8)
- added TP801: TestPoint, DIYPie:TestPoint_Pad_D1.5mm, F.Cu at (199.7, 34.4)
- added TP802: TestPoint, DIYPie:TestPoint_Pad_D1.5mm, F.Cu at (189.2, 41.4)
- added TP901: TestPoint, DIYPie:TestPoint_Pad_D1.5mm, F.Cu at (105.3, 115.5)
- added TP902: TestPoint, DIYPie:TestPoint_Pad_D1.5mm, F.Cu at (117.5, 92.8)
- added TP903: TestPoint, DIYPie:TestPoint_Pad_D1.5mm, F.Cu at (105.3, 111.9)
- added TP904: TestPoint, DIYPie:TestPoint_Pad_D1.5mm, F.Cu at (121.0, 92.8)
- added U10: DT1446-04V-7, DIYPie:SOT-563, F.Cu at (209.5, 102.3)
- added U1001: TLV320AIC3110IRHB, DIYPie:TI_TLV320AIC3110, F.Cu at (71.3, 105.8)
- added U1101: TPS61176, DIYPie:TI_TPS61176RTE, F.Cu at (146.6, 35.3)
- added U1201: TPS65132W, DIYPie:TI_TPS65132WRVC, F.Cu at (103.3, 35.8)
- added U1501: MIC94305, DIYPie:TDFN1616-6LD-PL-1, F.Cu at (170.5, 155.0)
- added U1601: MAX17260SETD+, DIYPie:MAXIM_TDFN-14-EP-T1433-2C, F.Cu at (292.4, 41.9)
- added U1701: AP7342, DIYPie:DIODES_X2-DFN1212-6, F.Cu at (195.7, 92.4)
- added U1801: TPS61023, DIYPie:SOT-563, F.Cu at (161.1, 151.3)
- added U201: TPS61176, DIYPie:TI_TPS61176RTE, F.Cu at (237.5, 63.6)
- added U202: TPS65132W, DIYPie:TI_TPS65132WRVC, F.Cu at (233.5, 78.4)
- added U2101: ATmega808-M, DIYPie:MICROCHIP_VQFN-32_RXB, F.Cu at (194.0, 118.8)
- added U401: TLV320AIC3110IRHB, DIYPie:TI_TLV320AIC3110, F.Cu at (137.4, 153.1)
- added U402: AP7342, DIYPie:DIODES_X2-DFN1212-6, F.Cu at (43.3, 181.9)
- added U5: ATmega808-M, DIYPie:MICROCHIP_VQFN-32_RXB, F.Cu at (32.0, 164.2)
- added U6: BQ24259RGE, DIYPie:TI_BQ24259RGE, F.Cu at (44.9, 163.7)
- added U7: MAX17260SETD+, DIYPie:MAXIM_TDFN-14-EP-T1433-2C, F.Cu at (32.1, 179.4)
- added U8: BQ24259RGE, DIYPie:TI_BQ24259RGE, F.Cu at (266.7, 51.8)
- added U9: FUSB303BTMX, DIYPie:ON_X2QFN-12_1.6x1.6mm_P0.4mm, F.Cu at (209.8, 117.1)
- added XA301: CM4, DIYPie:CM4_LOW_PROFILE_NoHoles, F.Cu at (37.4, 60.8)
- added Y1: 32K768, DIYPie:WE_830050789, F.Cu at (18.6, 185.6)
- added Y2101: 32K768, DIYPie:WE_830050789, F.Cu at (192.3, 124.0)
- C1: value 1u -> 470n; footprint DIYPie:C_0402_1005Metric_InvertedHomeplate -> DIYPie:C_0402_1005Metric
- C10, C5: value 4u7 -> 1u; footprint DIYPie:C_0603_1608Metric_InvertedHomeplate -> DIYPie:C_0402_1005Metric
- C11: value 4u7 -> 220p; footprint DIYPie:C_0805_2012Metric_InvertedHomeplate -> DIYPie:C_0402_1005Metric
- C12: value 1u -> 4u7; footprint DIYPie:C_0402_1005Metric_InvertedHomeplate -> DIYPie:C_0603_1608Metric
- C13, C14, C2: value 1u -> 10u; footprint DIYPie:C_0402_1005Metric_InvertedHomeplate -> DIYPie:C_0603_1608Metric
- C3: value 1u -> 220p; footprint DIYPie:C_0402_1005Metric_InvertedHomeplate -> DIYPie:C_0402_1005Metric
- C4: footprint DIYPie:C_0402_1005Metric_InvertedHomeplate -> DIYPie:C_0402_1005Metric
- C6: value 2u2 -> 1u; footprint DIYPie:C_0603_1608Metric_InvertedHomeplate -> DIYPie:C_0402_1005Metric
- C7: value 2u2 -> 12p; footprint DIYPie:C_0603_1608Metric_InvertedHomeplate -> DIYPie:C_0402_1005Metric
- C8: value 4u7 -> 12p; footprint DIYPie:C_0603_1608Metric_InvertedHomeplate -> DIYPie:C_0402_1005Metric
- C9: value 4u7 -> 47n; footprint DIYPie:C_0603_1608Metric_InvertedHomeplate -> DIYPie:C_0402_1005Metric
- D1: value PMEG4010CEJ -> DF2B7AFS; footprint DIYPie:D_SOD-323F -> DIYPie:D_SOD-923
- D2: value STATUS_LED -> STATUS; footprint DIYPie:KINGBRIGHT_APFA3010 -> DIYPie:KINGBRIGHT_APBA3010
- J1: value DF40C-100DS-0.4V(51) -> SPK_L; footprint DIYPie:hirose_DF40C-100DS-0.4V(51)_NoPads -> DIYPie:MOLEX_533980267
- J2: value DF40C-100DS-0.4V(51) -> BAT; footprint DIYPie:hirose_DF40C-100DS-0.4V(51)_NoPads -> DIYPie:MOLEX_533980267
- J3: value CUI_DEVICES_SJ-43514-SMT -> MOLEX_2171790001; footprint DIYPie:CUI_DEVICES_SJ-43514-SMT -> DIYPie:MOLEX_2171790001
- J4: value MOLEX_5033981892 -> MOLEX_2171790001; footprint DIYPie:MOLEX_5033981892 -> DIYPie:MOLEX_2171790001
- L1: value 4u7 -> 1u; footprint DIYPie:L_0805_2012Metric_InvertedHomeplate -> DIYPie:L_TYA4020
- L2: value 4u7 -> 1u; footprint DIYPie:L_1008_2520Metric_InvertedHomeplate -> DIYPie:L_TYA4020
- R1: value 34K -> 100R; footprint DIYPie:R_0402_1005Metric_InvertedHomeplate -> DIYPie:R_0402_1005Metric
- R3: value 732K -> 10K; footprint DIYPie:R_0402_1005Metric_InvertedHomeplate -> DIYPie:R_0402_1005Metric
- R4: value 34K -> 732K; footprint DIYPie:R_0402_1005Metric_InvertedHomeplate -> DIYPie:R_0402_1005Metric
- SW2: value VOL_UP -> VOL+
- SW3: value VOL_DOWN -> VOL-
- U1: value TPS65132W -> TPS61023; footprint DIYPie:TI_TPS65132WRVC -> DIYPie:SOT-563
- U2: value TPS61176 -> MIC94305; footprint DIYPie:TI_TPS61176RTE -> DIYPie:TDFN1616-6LD-PL-1
- U3: value TPS61023 -> FUSB303BTMX; footprint DIYPie:SOT-563 -> DIYPie:ON_X2QFN-12_1.6x1.6mm_P0.4mm
- U4: value TLV320AIC3110IRHB -> DT1446-04V-7; footprint DIYPie:TI_TLV320AIC3110 -> DIYPie:SOT-563
- moved R1 172.8 mm to (241.2, 92.5)
- moved SW1 159.1 mm to (228.7, 101.9), turned to 0 degrees
- moved SW3 155.8 mm to (234.9, 94.7), turned to 0 degrees
- moved D2 154.3 mm to (229.2, 107.7), turned to 0 degrees
- moved SW2 142.1 mm to (228.7, 94.7), turned to 0 degrees
- moved J3 119.3 mm to (22.5, 165.6)
- moved J2 117.9 mm to (21.9, 172.8)
- moved J4 100.0 mm to (213.7, 96.1)
- moved C12 65.1 mm to (29.7, 183.7)
- moved C4 60.5 mm to (37.1, 185.5)
- moved U4 55.9 mm to (32.5, 183.6)
- moved C8 52.3 mm to (41.0, 182.0)
- moved L1 51.3 mm to (25.6, 184.0)
- moved R3 51.1 mm to (40.8, 176.1)
- moved C10 47.8 mm to (43.0, 179.0)
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Connections:
- C1 pad 1: Net-(C1-Pad1) -> +3V3
- C10 pad 1: /Display/lcm_avee -> GND
- C10 pad 2: GND -> +3V3
- C11 pad 1: /Display/lcm_led+ -> GND
- C11 pad 2: GND -> /System Control Block/scb_usb_cc2
- C12 pad 1: +1V8 -> Net-(C12-Pad1)
- C13 pad 1: +3V3 -> Net-(C13-Pad1)
- C14 pad 1: +1V8 -> +5V
- C2 pad 1: +3V3 -> Net-(C2-Pad1)
- C3 pad 1: Net-(C3-Pad1) -> GND
- C3 pad 2: GND -> /System Control Block/scb_usb_cc1
- C4 pad 1: +3V3 -> GND
- C4 pad 2: GND -> +3V3
- C5 pad 1: +BATT -> GND
- C5 pad 2: GND -> +3V3
- C6 pad 1: +BATT -> GND
- C6 pad 2: GND -> +5V
- C7 pad 2: Net-(C7-Pad2) -> GND
- C8 pad 1: /Display/lcm_avdd -> Net-(C8-Pad1)
- C9 pad 2: GND -> Net-(C9-Pad2)
- D1 pad 1: /Display/lcm_led+ -> Net-(D1-Pad1)
- D1 pad 2: Net-(D1-Pad2) -> GND
- D2 pad 1: (no net) -> +3V3
- D2 pad 2: (no net) -> Net-(D2-Pad2)
- D2 pad 3: (no net) -> Net-(D2-Pad3)
- L1 pad 1: Net-(L1-Pad1) -> Net-(C9-Pad1)
- L1 pad 2: +BATT -> +5V
- L2 pad 1: +BATT -> +5V
- L2 pad 2: Net-(D1-Pad2) -> Net-(L2-Pad2)
- R1 pad 1: Net-(R1-Pad1) -> /Buttons & LEDs/scb_led_r
- R1 pad 2: GND -> Net-(D2-Pad2)
- R3 pad 1: /Display/lcm_led+ -> +3V3
- R3 pad 2: Net-(R3-Pad2) -> /System Control Block/scb_int_usbc
- R4 pad 1: Net-(R3-Pad2) -> Net-(R4-Pad1)
- SW1 pad 1: (no net) -> GND
- SW1 pad 2: (no net) -> /Buttons & LEDs/scb_sw_pow
- SW1 pad 3: (no net) -> GND
- SW1 pad MP: Net-(SW1-PadMP) -> GND
- SW2 pad 1: (no net) -> GND
- SW2 pad 2: (no net) -> /Buttons & LEDs/scb_sw_vol+
- SW2 pad 3: (no net) -> GND
- SW2 pad MP: Net-(SW2-PadMP) -> GND
- SW3 pad 1: (no net) -> GND
- SW3 pad 2: (no net) -> /Buttons & LEDs/scb_sw_vol-
- SW3 pad 3: (no net) -> GND
- SW3 pad MP: Net-(SW3-PadMP) -> GND
- U1 pad 1: GND -> Net-(C19-Pad1)
- U1 pad 2: GND -> /System Control Block/scb_5v_en
- U1 pad 3: GND -> +5V
- U1 pad 4: +3V3 -> GND
- U1 pad 5: (no net) -> Net-(L2-Pad2)
- U1 pad 6: (no net) -> +5V
- U2 pad 1: /Display/lcm_ledpwm -> Net-(C2-Pad1)
- U2 pad 2: Net-(C1-Pad1) -> Net-(C2-Pad1)
- U2 pad 3: Net-(R1-Pad1) -> GND
- U2 pad 4: Net-(C3-Pad1) -> /Memory/mem_pwr
- U2 pad 5: GND -> +3V3
- U2 pad 6: GND -> +3V3
- U2 pad 7: /Display/lcm_led2- -> GND
- U3 pad 1: (no net) -> /System Control Block/scb_usb_cc1
- U3 pad 2: (no net) -> /System Control Block/scb_usb_cc2
- U3 pad 3: (no net) -> unconnected-(U3-Pad3)
- U3 pad 4: (no net) -> +5V
- U3 pad 5: (no net) -> Net-(R4-Pad1)
- U3 pad 6: (no net) -> /System Control Block/scb_int_usbc
- U4 pad 1: GND -> /System Control Block/scb_usb_dm
- U4 pad 2: +3V3 -> GND
- U4 pad 3: +1V8 -> /System Control Block/scb_usb_cc2
- U4 pad 4: (no net) -> /System Control Block/scb_usb_dp
- U4 pad 5: (no net) -> +5V
- U4 pad 6: (no net) -> /System Control Block/scb_usb_cc1
Routing:
- net /Headpnones/MIC: track 0.00 -> 21.9 mm
Other:
- board outline removed
- net class Default removed
